File: DAB_Pablo/Primary Side Half-Bridge 2.kicad_sch (KiCad schematic)
At the start: 89 parts, among them U32 UCC14141QDWNRQ1, U33 UCC14141QDWNRQ1, U37 UCC21710QDWQ1, U38 UCC21710QDWQ1

Commit message: Se finaliza todos los half-bridge
Parts:
- renumbered C112 to C237, C113 to C238, C149 to C275, C150 to C276, C236 to C277, C242 to C278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
