File: DAB_Pablo/Secondary Side Half-Bridge 1.kicad_sch (KiCad schematic)
At the start: 89 parts, among them U32 UCC14141QDWNRQ1, U33 UCC14141QDWNRQ1, U37 UCC21710QDWQ1, U38 UCC21710QDWQ1

Commit message: Se finaliza todos los half-bridge
Parts:
- renumbered C248 to C196, C149 to C198, C150 to C199, C112 to C200, C113 to C201, C236 to C202, C232 to C203, C242 to C204, C243 to C205, C240 to C206, C82 to C207, C246 to C208, C247 to C209, C244 to C210, C245 to C211, C249 to C212, C250 to C213, C251 to C214, C252 to C215, C253 to C216, C254 to C217, C255 to C218, C256 to C219, C257 to C220, C258 to C221, C259 to C222, C260 to C223, C261 to C224, C262 to C225, C264 to C226, C265 to C227, C266 to C228, C268 to C229, C269 to C230, C270 to C231, C274 to C233, C298 to C234, C302 to C235, C330 to C327, C329 to C328, C94 to C88, D26 to D18, D22 to D19, D32 to D21, D31 to D8, R18 to R17, R210 to R193, R211 to R194, R212 to R206, R213 to R207, R288 to R241, R291 to R243, R292 to R244, R286 to R245, R293 to R246, R294 to R247, R287 to R248, R289 to R249, R290 to R250, R301 to R255, R302 to R256, R298 to R257, R299 to R258, R303 to R259, R32 to R26, R304 to R260, R306 to R260, R305 to R261, R311 to R267, R316 to R272, R317 to R273, R318 to R274, R316 to R275, R320 to R276, R321 to R277, R322 to R278, R323 to R279, R324 to R280, R325 to R282, R326 to R284, R31 to R78, R11 to R9, R130 to R94, R104 to R99, RT3 to RT2, U33 to U27, U32 to U28, U37 to U34, U38 to U35
Connections:
- net +15V_BOT2 renamed +15V_BOT3
- net +15V_TOP2 renamed +15V_TOP3
- net -4V_BOT2 renamed -4V_BOT3
- net -4V_TOP2 renamed -4V_TOP3
- net GND_BOT2 renamed GND_BOT3
- net GND_TOP2 renamed GND_TOP3
Other:
- note added: "Secondary Side Half-Bridge 1"
- note removed: "Primary Side Half-Bridge 2"
