File: DAB_Pablo/Secondary Side Half-Bridge 2.kicad_sch (KiCad schematic)
At the start: 89 parts, among them U32 UCC14141QDWNRQ1, U33 UCC14141QDWNRQ1, U37 UCC21710QDWQ1, U38 UCC21710QDWQ1

Commit message: Se finaliza todos los half-bridge
Connections:
- net +15V_BOT2 renamed +15V_BOT4
- net +15V_TOP2 renamed +15V_TOP4
- net -4V_BOT2 renamed -4V_BOT4
- net -4V_TOP2 renamed -4V_TOP4
- net GND_BOT2 renamed GND_BOT4
- net GND_TOP2 renamed GND_TOP4
Other:
- note added: "Secondary Side Half-Bridge 2"
- note removed: "Primary Side Half-Bridge 2"
