File: DAB_Pablo/untitled.kicad_sch (KiCad schematic)
At the start: 89 parts, among them U1 UCC14141QDWNRQ1, U2 UCC21710QDWQ1, U3 UCC14141QDWNRQ1, U4 UCC21710QDWQ1

Commit message: Se finaliza todos los half-bridge
Parts:
- R8: renamed from R34; value 1.0k -> 604
- renumbered C2 to C155, C5 to C156, C23 to C157, C26 to C158, C9 to C159, C30 to C160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
Connections:
- net TMP_HB1_P: no longer U30.16 (APWM)
